File: MotorDriver/MotorDriver.kicad_pcb (KiCad board)
At the start: 2 copper layers, 56 x 54 mm, 85 parts, among them J1 Screw_Terminal_01x04, J2 Screw_Terminal_01x04, Q1 BSS84, Q2 2N7002, Q3 BSS84, Q4 2N7002, Q5 2N7002, Q6 2N7002, Q7 2N7002, U1 DRV8251ADDAR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

Commit message: Add LCSC order numbers
Parts:
- R11, R12, R14, R2: value 27K -> 33K
- R18: value 22K -> 33K
- R19: value 120K -> 180K
Changed lines of the file:
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@@
     (descr "SOT, 3 Pin (https://www.jedec.org/system/files/docs/to-236h.pdf variant AB), generated with kicad-footprint-generator ipc_gullwing_generator.py")
     (tags "SOT TO_SOT_SMD")
+    (property "LCSC" "C65189")
     (property "Sheetfile" "MotorDriver.kicad_sch")
     (property "Sheetname" "")
@@
     (descr "SOT, 3 Pin (https://www.jedec.org/system/files/docs/to-236h.pdf variant AB), generated with kicad-footprint-generator ipc_gullwing_generator.py")
     (tags "SOT TO_SOT_SMD")
+    (property "LCSC" "C65189")
     (property "Sheetfile" "MotorDriver.kicad_sch")
     (property "Sheetname" "")
@@
         (effects (font (size 0.9 0.8) (thickness 0.15)))
     )
-    (fp_text value "27K" (at 0 1.43) (layer "F.Fab")
+    (fp_text value "33K" (at 0 1.43) (layer "F.Fab")
         (effects (font (size 1 1) (thickness 0.15)))
     )
@@
     (descr "SOD-123")
     (tags "SOD-123")
+    (property "LCSC" "C85181")
     (property "Ordercode" "MMSZ4689-TP")
     (property "Sheetfile" "MotorDriver.kicad_sch")
@@
     (descr "LED SMD 0603 (1608 Metric), square (rectangular) end terminal, IPC_7351 nominal, (Body size source: http://www.tortai-tech.com/upload/download/2011102023233369053.pdf), generated with kicad-footprint-generator")
     (tags "LED")
+    (property "LCSC" "C965799")
     (property "Sheetfile" "MotorDriver.kicad_sch")
     (property "Sheetname" "")
@@
     (descr "Potentiometer, Bourns, TC33X, Vertical, https://www.bourns.com/pdfs/TC33.pdf")
     (tags "Potentiometer Bourns TC33X Vertical")
+    (property "LCSC" "C6331330")
     (property "Sheetfile" "MotorDriver.kicad_sch")
     (property "Sheetname" "")
@@
     (descr "SOD-123")
     (tags "SOD-123")
+    (property "LCSC" "C19077504")
     (property "Sheetfile" "MotorDriver.kicad_sch")
     (property "Sheetname" "")
@@
     (at 180.77365 92.6 -90)
     (tags "TLV709A01DBVR ")
+    (property "LCSC" "C22365366")
     (property "Sheetfile" "MotorDriver.kicad_sch")
     (property "Sheetname" "")
@@
     (descr "SOT, 3 Pin (https://www.jedec.org/system/files/docs/to-236h.pdf variant AB), generated with kicad-footprint-generator ipc_gullwing_generator.py")
     (tags "SOT TO_SOT_SMD")
+    (property "LCSC" "C82079")
     (property "Sheetfile" "MotorDriver.kicad_sch")
     (property "Sheetname" "")
@@
         (effects (font (size 0.9 0.8) (thickness 0.15)))
     )
-    (fp_text value "27K" (at 0 1.43) (layer "F.Fab")
+    (fp_text value "33K" (at 0 1.43) (layer "F.Fab")
         (effects (font (size 1 1) (thickness 0.15)))
     )
@@
     (descr "SOT, 3 Pin (https://www.jedec.org/system/files/docs/to-236h.pdf variant AB), generated with kicad-footprint-generator ipc_gullwing_generator.py")
     (tags "SOT TO_SOT_SMD")
+    (property "LCSC" "C65189")
     (property "Sheetfile" "MotorDriver.kicad_sch")
     (property "Sheetname" "")
@@
     (descr "Potentiometer, Bourns, TC33X, Vertical, https://www.bourns.com/pdfs/TC33.pdf")
     (tags "Potentiometer Bourns TC33X Vertical")
+    (property "LCSC" "C6331330")
     (property "Sheetfile" "MotorDriver.kicad_sch")
     (property "Sheetname" "")
@@
     (at 148.25 96.975 90)
     (tags "DRV8251ADDAR ")
+    (property "LCSC" "C5218844")
     (property "Sheetfile" "MotorDriver.kicad_sch")
     (property "Sheetname" "")
@@
         (effects (font (size 1 1) (thickness 0.15)))
     )
-    (fp_text user "*" (at -1.6129 -2.4257 90) (layer "F.Fab")
+    (fp_text user "*" (at -1.6129 -2.4257 90 unlocked) (layer "F.Fab")
         (effects (font (size 1 1) (thickness 0.15)))
     )
-    (fp_text user "${REFERENCE}" (at 0 0 90 unlocked) (layer "F.Fab")
+    (fp_text user "*" (at -1.6129 -2.4257 90) (layer "F.Fab")
         (effects (font (size 1 1) (thickness 0.15)))
     )
-    (fp_text user "*" (at -1.6129 -2.4257 90 unlocked) (layer "F.Fab")
+    (fp_text user "${REFERENCE}" (at 0 0 90 unlocked) (layer "F.Fab")
         (effects (font (size 1 1) (thickness 0.15)))
     )
@@
     (descr "SOT, 3 Pin (https://www.jedec.org/system/files/docs/to-236h.pdf variant AB), generated with kicad-footprint-generator ipc_gullwing_generator.py")
     (tags "SOT TO_SOT_SMD")
+    (property "LCSC" "C65189")
     (property "Sheetfile" "MotorDriver.kicad_sch")
     (property "Sheetname" "")
@@
     (descr "Diode SMA (DO-214AC)")
     (tags "SMA (DO-214AC)")
+    (property "LCSC" "C1974908")
     (property "Sheetfile" "MotorDriver.kicad_sch")
     (property "Sheetname" "")
@@
     (descr "SMD capacitor, aluminum electrolytic, Nichicon, 8.0x10mm")
     (tags "capacitor electrolytic")
+    (property "LCSC" "C278406")
     (property "Sheetfile" "MotorDriver.kicad_sch")
     (property "Sheetname" "")
@@
     (descr "Diode SMA (DO-214AC)")
     (tags "SMA (DO-214AC)")
+    (property "LCSC" "C1974908")
     (property "Sheetfile" "MotorDriver.kicad_sch")
     (property "Sheetname" "")
@@
         (effects (font (size 0.9 0.8) (thickness 0.15)))
     )
-    (fp_text value "27K" (at 0 1.43 90) (layer "F.Fab")
+    (fp_text value "33K" (at 0 1.43 90) (layer "F.Fab")
         (effects (font (size 1 1) (thickness 0.15)))
     )
@@
     (descr "SOD-123")
     (tags "SOD-123")
+    (property "LCSC" "C19077504")
     (property "Sheetfile" "MotorDriver.kicad_sch")
     (property "Sheetname" "")
@@
     (descr "SOIC, 8 Pin (JEDEC MS-012AA, https://www.analog.com/media/en/package-pcb-resources/package/pkg_pdf/soic_narrow-r/r_8.pdf), generated with kicad-footprint-generator ipc_gullwing_generator.py")
     (tags "SOIC SO")
+    (property "LCSC" "C90760")
     (property "Sheetfile" "MotorDriver.kicad_sch")
     (property "Sheetname" "")
@@
         (effects (font (size 0.9 0.8) (thickness 0.15)))
     )
-    (fp_text value "22K" (at 0 1.43 -270) (layer "F.Fab")
+    (fp_text value "33K" (at 0 1.43 -270) (layer "F.Fab")
         (effects (font (size 1 1) (thickness 0.15)))
     )
@@
     (descr "Diode SMA (DO-214AC)")
     (tags "SMA (DO-214AC)")
+    (property "LCSC" "C1974908")
     (property "Sheetfile" "MotorDriver.kicad_sch")
     (property "Sheetname" "")
@@
         (effects (font (size 0.9 0.8) (thickness 0.15)))
     )
-    (fp_text value "27K" (at 0 1.43) (layer "F.Fab")
+    (fp_text value "33K" (at 0 1.43) (layer "F.Fab")
         (effects (font (size 1 1) (thickness 0.15)))
     )
@@
         (effects (font (size 0.9 0.8) (thickness 0.15)))
     )
-    (fp_text value "120K" (at 0 1.43) (layer "F.Fab")
+    (fp_text value "180K" (at 0 1.43) (layer "F.Fab")
         (effects (font (size 1 1) (thickness 0.15)))
     )
@@
     (at 140.25 105.25 -90)
     (tags "AP331AWG-7 ")
+    (property "LCSC" "C151034")
     (property "Sheetfile" "MotorDriver.kicad_sch")
     (property "Sheetname" "")
@@
     (descr "SMD capacitor, aluminum electrolytic, Nichicon, 8.0x10mm")
     (tags "capacitor electrolytic")
+    (property "LCSC" "C278406")
     (property "Sheetfile" "MotorDriver.kicad_sch")
     (property "Sheetname" "")
@@
     (descr "SOT, 3 Pin (https://www.jedec.org/system/files/docs/to-236h.pdf variant AB), generated with kicad-footprint-generator ipc_gullwing_generator.py")
     (tags "SOT TO_SOT_SMD")
+    (property "LCSC" "C65189")
     (property "Sheetfile" "MotorDriver.kicad_sch")
     (property "Sheetname" "")
@@
     (descr "LED SMD 0603 (1608 Metric), square (rectangular) end terminal, IPC_7351 nominal, (Body size source: http://www.tortai-tech.com/upload/download/2011102023233369053.pdf), generated with kicad-footprint-generator")
     (tags "LED")
+    (property "LCSC" "C5656657")
     (property "Sheetfile" "MotorDriver.kicad_sch")
     (property "Sheetname" "")
@@
     (descr "Potentiometer, Bourns, TC33X, Vertical, https://www.bourns.com/pdfs/TC33.pdf")
     (tags "Potentiometer Bourns TC33X Vertical")
+    (property "LCSC" "C6331330")
     (property "Sheetfile" "MotorDriver.kicad_sch")
     (property "Sheetname" "")
@@
     (descr "SOD-123")
     (tags "SOD-123")
+    (property "LCSC" "C19077504")
     (property "Sheetfile" "MotorDriver.kicad_sch")
     (property "Sheetname" "")
@@
     (descr "LED SMD 0603 (1608 Metric), square (rectangular) end terminal, IPC_7351 nominal, (Body size source: http://www.tortai-tech.com/upload/download/2011102023233369053.pdf), generated with kicad-footprint-generator")
     (tags "LED")
+    (property "LCSC" "C5656657")
     (property "Sheetfile" "MotorDriver.kicad_sch")
     (property "Sheetname" "")
@@
     (descr "SOT, 3 Pin (https://www.jedec.org/system/files/docs/to-236h.pdf variant AB), generated with kicad-footprint-generator ipc_gullwing_generator.py")
     (tags "SOT TO_SOT_SMD")
+    (property "LCSC" "C82079")
     (property "Sheetfile" "MotorDriver.kicad_sch")
     (property "Sheetname" "")
