File: MotorDriver/MotorDriver.kicad_sch (KiCad schematic)
At the start: 84 parts, among them J1 Screw_Terminal_01x04, J2 Screw_Terminal_01x04, Q1 BSS84, Q2 2N7002, Q3 BSS84, Q4 2N7002, Q5 2N7002, Q6 2N7002, Q7 2N7002, U1 DRV8251ADDAR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

Commit message: Add LCSC order numbers
Parts:
- C3, C4: LCSC (none) -> C278406
- D1, D3: LCSC (none) -> C5656657
- D10, D6, D7: LCSC (none) -> C19077504
- D2: LCSC (none) -> C85181
- D4: LCSC (none) -> C965799
- D5, D8, D9: LCSC (none) -> C1974908
- Q1, Q3: LCSC (none) -> C82079
- Q2, Q4, Q5, Q6, Q7: LCSC (none) -> C65189
- R11, R12, R14, R2: value 27K -> 33K
- R18: value 22K -> 33K
- R19: value 120K -> 180K
- RV1, RV2, RV3: LCSC (none) -> C6331330
- U1: LCSC (none) -> C5218844
- U2: LCSC (none) -> C151034
- U3: LCSC (none) -> C90760
- U4: LCSC (none) -> C22365366
Other:
- note added: "Min. button release time before resetting latch: approx. 33e3 * 10e-6 = 330 ms"
- note added: "Open source hardware © 2024 Anthony Bernaert Licensed under CERN-OHL-P v2"
- note removed: "Min. button release time before resetting latch: approx. 27e3 * 10e-6 = 270 ms"
- title: (none) -> DC motor driver with stall detection
Changed lines of the file:
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@@
   (paper "A3")
   (title_block
+    (title "DC motor driver with stall detection")
+    (date "2024-12-02")
     (rev "1")
   )
@@
     (effects (font (size 2 2)) (justify left bottom))
   )
-  (text "Min. button release time before resetting latch:\napprox. 27e3 * 10e-6 = 270 ms"
+  (text "Min. button release time before resetting latch:\napprox. 33e3 * 10e-6 = 330 ms"
     (at 147.32 190.5 0)
     (effects (font (size 1.27 1.27)) (justify left bottom))
@@
     (effects (font (size 2 2)) (justify left bottom))
   )
+  (text "Open source hardware\n\n© 2024 Anthony Bernaert\nLicensed under CERN-OHL-P v2"
+    (at 318.135 266.065 0)
+    (effects (font (size 1.8 1.8)) (justify left bottom))
+  )
   (text "Motor stall detection + latch" (at 127 135.89 0)
     (effects (font (size 2 2)) (justify left bottom))
@@
       (effects (font (size 1.27 1.27)) (justify left) hide)
     )
+    (property "LCSC" "C65189" (at 363.855 165.1 0)
+      (effects (font (size 1.27 1.27)) hide)
+    )
     (pin "1")
     (pin "2")
@@
       (effects (font (size 1.27 1.27)) (justify left))
     )
-    (property "Value" "27K" (at 213.36 154.305 0)
+    (property "Value" "33K" (at 213.36 154.305 0)
       (effects (font (size 1.27 1.27)) (justify left))
     )
@@
       (effects (font (size 1.27 1.27)) hide)
     )
+    (property "LCSC" "C19077504" (at 296.545 205.105 90)
+      (effects (font (size 1.27 1.27)) hide)
+    )
     (pin "1")
     (pin "2")
@@
       (effects (font (size 1.27 1.27)) hide)
     )
+    (property "LCSC" "C6331330" (at 151.13 157.48 90)
+      (effects (font (size 1.27 1.27)) hide)
+    )
     (pin "1")
     (pin "2")
@@
       (effects (font (size 1.27 1.27)) (justify left))
     )
-    (property "Value" "22K" (at 180.34 95.885 0)
+    (property "Value" "33K" (at 180.34 95.885 0)
       (effects (font (size 1.27 1.27)) (justify left))
     )
@@
       (effects (font (size 1.27 1.27)))
     )
-    (property "Value" "LED AMBER" (at 334.01 175.26 0)
+    (property "Value" "LED AMBER" (at 330.835 175.26 0)
       (effects (font (size 1.27 1.27)))
     )
@@
       (effects (font (size 1.27 1.27)) hide)
     )
+    (property "LCSC" "C5656657" (at 335.28 168.91 0)
+      (effects (font (size 1.27 1.27)) hide)
+    )
     (pin "1")
     (pin "2")
@@
       (effects (font (size 1.27 1.27) italic) hide)
     )
+    (property "LCSC" "C5218844" (at 283.21 82.55 0)
+      (effects (font (size 1.27 1.27)) hide)
+    )
     (pin "2")
     (pin "3")
@@
       (effects (font (size 1.27 1.27)) hide)
     )
+    (property "LCSC" "C85181" (at 252.73 97.79 90)
+      (effects (font (size 1.27 1.27)) hide)
+    )
     (pin "1")
     (pin "2")
@@
       (effects (font (size 1.27 1.27)) hide)
     )
+    (property "LCSC" "C19077504" (at 254.635 211.455 90)
+      (effects (font (size 1.27 1.27)) hide)
+    )
     (pin "1")
     (pin "2")
@@
       (effects (font (size 1.27 1.27)) hide)
     )
+    (property "LCSC" "C278406" (at 354.33 97.79 0)
+      (effects (font (size 1.27 1.27)) hide)
+    )
     (pin "1")
     (pin "2")
@@
       (effects (font (size 1.27 1.27)) (justify left) hide)
     )
+    (property "LCSC" "C65189" (at 238.76 210.82 0)
+      (effects (font (size 1.27 1.27)) hide)
+    )
     (pin "1")
     (pin "2")
@@
       (effects (font (size 1.27 1.27)) (justify left) hide)
     )
+    (property "LCSC" "C65189" (at 152.4 199.39 0)
+      (effects (font (size 1.27 1.27)) hide)
+    )
     (pin "1")
     (pin "2")
@@
       (effects (font (size 1.27 1.27)) hide)
     )
+    (property "LCSC" "C19077504" (at 300.99 163.195 90)
+      (effects (font (size 1.27 1.27)) hide)
+    )
     (pin "1")
     (pin "2")
@@
       (effects (font (size 1.27 1.27)) (justify left) hide)
     )
+    (property "LCSC" "C82079" (at 320.04 154.94 0)
+      (effects (font (size 1.27 1.27)) hide)
+    )
     (pin "1")
     (pin "2")
@@
       (effects (font (size 1.27 1.27)) hide)
     )
+    (property "LCSC" "C278406" (at 347.98 97.79 0)
+      (effects (font (size 1.27 1.27)) hide)
+    )
     (pin "1")
     (pin "2")
@@
       (effects (font (size 1.27 1.27)) (justify left) hide)
     )
+    (property "LCSC" "C65189" (at 179.07 199.39 0)
+      (effects (font (size 1.27 1.27)) hide)
+    )
     (pin "1")
     (pin "2")
@@
       (effects (font (size 1.27 1.27)) hide)
     )
+    (property "LCSC" "C1974908" (at 368.3 97.79 90)
+      (effects (font (size 1.27 1.27)) hide)
+    )
     (pin "1")
     (pin "2")
@@
       (effects (font (size 1.27 1.27)) hide)
     )
+    (property "LCSC" "C6331330" (at 245.11 97.79 0)
+      (effects (font (size 1.27 1.27)) hide)
+    )
     (pin "1")
     (pin "2")
@@
       (effects (font (size 1.27 1.27)) hide)
     )
+    (property "LCSC" "C90760" (at 185.42 162.56 0)
+      (effects (font (size 1.27 1.27)) hide)
+    )
     (pin "1")
     (pin "8")
@@
       (effects (font (size 1.27 1.27)) (justify left))
     )
-    (property "Value" "27K" (at 238.76 81.28 0)
+    (property "Value" "33K" (at 238.76 81.28 0)
       (effects (font (size 1.27 1.27)) (justify left))
     )
@@
       (effects (font (size 1.27 1.27)) hide)
     )
+    (property "LCSC" "C1974908" (at 88.9 80.01 90)
+      (effects (font (size 1.27 1.27)) hide)
+    )
     (pin "1")
     (pin "2")
@@
       (effects (font (size 1.27 1.27)) (justify left))
     )
-    (property "Value" "27K" (at 134.62 149.86 0)
+    (property "Value" "33K" (at 134.62 149.86 0)
       (effects (font (size 1.27 1.27)) (justify left))
     )
@@
       (effects (font (size 1.27 1.27)))
     )
-    (property "Value" "LED AMBER" (at 334.01 215.9 0)
+    (property "Value" "LED AMBER" (at 330.2 215.9 0)
       (effects (font (size 1.27 1.27)))
     )
@@
       (effects (font (size 1.27 1.27)) hide)
     )
+    (property "LCSC" "C5656657" (at 335.28 209.55 0)
+      (effects (font (size 1.27 1.27)) hide)
+    )
     (pin "1")
     (pin "2")
@@
       (effects (font (size 1.27 1.27)) (justify left) hide)
     )
+    (property "LCSC" "C65189" (at 363.855 205.74 0)
+      (effects (font (size 1.27 1.27)) hide)
+    )
     (pin "1")
     (pin "2")
@@
       (effects (font (size 1.27 1.27)))
     )
-    (property "Value" "27K" (at 260.35 167.64 90)
+    (property "Value" "33K" (at 260.35 167.64 90)
       (effects (font (size 1.27 1.27)))
     )
@@
       (effects (font (size 1.27 1.27)) (justify left) hide)
     )
+    (property "LCSC" "C82079" (at 320.04 195.58 0)
+      (effects (font (size 1.27 1.27)) hide)
+    )
     (pin "1")
     (pin "2")
@@
       (effects (font (size 1.27 1.27)) hide)
     )
+    (property "LCSC" "C965799" (at 240.03 171.45 90)
+      (effects (font (size 1.27 1.27)) hide)
+    )
     (pin "1")
     (pin "2")
@@
       (effects (font (size 1.27 1.27)) hide)
     )
+    (property "LCSC" "C1974908" (at 360.68 97.79 90)
+      (effects (font (size 1.27 1.27)) hide)
+    )
     (pin "1")
     (pin "2")
@@
       (effects (font (size 1.27 1.27)) (justify left))
     )
-    (property "Value" "120K" (at 176.53 85.725 0)
+    (property "Value" "180K" (at 176.53 85.725 0)
       (effects (font (size 1.27 1.27)) (justify left))
     )
@@
       (effects (font (size 1.27 1.27) italic) hide)
     )
+    (property "LCSC" "C22365366" (at 131.445 78.74 0)
+      (effects (font (size 1.27 1.27)) hide)
+    )
     (pin "1")
     (pin "2")
@@
       (effects (font (size 1.27 1.27) italic) hide)
     )
+    (property "LCSC" "C151034" (at 55.88 153.67 0)
+      (effects (font (size 1.27 1.27)) hide)
+    )
     (pin "1")
     (pin "2")
@@
       (effects (font (size 1.27 1.27)) hide)
     )
+    (property "LCSC" "C6331330" (at 135.89 167.64 0)
+      (effects (font (size 1.27 1.27)) hide)
+    )
     (pin "1")
     (pin "2")
@@
         )
       )
+    )
+  )
+  (symbol (lib_id "Graphic:Logo_Open_Hardware_Small") (at 309.245 260.985 0) (unit 1)
+    (in_bom no) (on_board no) (dnp no) (fields_autoplaced)
+    (property "Reference" "#SYM5" (at 309.245 254 0)
+      (effects (font (size 1.27 1.27)) hide)
+    )
+    (property "Value" "Logo_Open_Hardware_Small" (at 309.245 266.7 0)
+      (effects (font (size 1.27 1.27)) hide)
+    )
+    (property "Footprint" "" (at 309.245 260.985 0)
+      (effects (font (size 1.27 1.27)) hide)
+    )
+    (property "Datasheet" "~" (at 309.245 260.985 0)
+      (effects (font (size 1.27 1.27)) hide)
+    )
+    (property "Sim.Enable" "0" (at 309.245 260.985 0)
+      (effects (font (size 1.27 1.27)) hide)
+    )
+    (instances
+      (project "MotorDriver"
+        (path "/e411bfac-3723-4745-962d-7c716bdbc4b1"
+          (reference "#SYM5") (unit 1)
+        )
+      )
